Commit message: second time

File: URDF/robot.urdf (robot description, URDF)
Before this commit: robot mobile_robot, 4 links, 3 joints
Links:
- added link dummy
- link base_link: mass None -> 2.5; geometry collision cylinder length=0.02 radius=0.15; visual cylinder length=0.02 radius=0.15
- link caster: mass None -> 2.5; geometry collision sphere radius=0.02; visual sphere radius=0.02
- link left_wheel: mass None -> 2.5; geometry collision cylinder length=0.02 radius=0.04; visual cylinder length=0.02 radius=0.04
- link right_wheel: mass None -> 2.5; geometry collision cylinder length=0.02 radius=0.04; visual cylinder length=0.02 radius=0.04
Joints:
- added joint dummy_joint: type fixed, parent dummy, child base_link
