Commit message: third commit

File: URDF/robot.xacro (robot description, xacro)
@@ -19,4 +19,15 @@
 <xacro:property name="caster_joint_y" value="0.12"/>
 <xacro:property name="caster_joint_z" value="0.02"/>
+<!--property of moment inertial-->
+<xacro:property name="mass" value="5"/>
+<xacro:property name="ixx" value="0.01"/>
+<xacro:property name="iyy" value="0.01"/>
+<xacro:property name="izz" value="0.01"/>
+<link name="dummy" >
+</link>
+<joint name="dummy_base_link" type="fixed">
+	<parent link="dummy"/>
+	<child link="base_link"/>
+</joint>
 <link name="base_link">
 	<visual>
@@ -26,4 +37,15 @@
 		</geometry>
 	</visual>
+	<collision>
+		<origin rpy="0 0 0" xyz="0 0 0"/>
+		<geometry>
+			<cylinder length="${base_link_length}" radius="${base_link_radius}" />
+		</geometry>
+	</collision>
+	<inertial>
+		<mass value="${mass}"/>
+		<origin xyz=" 0 0 0 "/>
+		<inertia ixx="${ixx}" ixy="0" ixz="0" iyy="${iyy}" iyz="0" izz="${izz}"/>
+	</inertial>
 </link>
 <link name="left_wheel">
@@ -34,4 +56,15 @@
 		</geometry>
 	</visual>
+	<collision>
+		<origin rpy="0 ${wheel_pitch} 0" xyz="0 0 0"/>
+		<geometry>
+			<cylinder length="${wheel_length}" radius="${wheel_radius}"/>
+		</geometry>
+	</collision>
+	<inertial>
+		<mass value="${mass}"/>
+		<origin xyz=" 0 0 0 "/>
+		<inertia ixx="${ixx}" ixy="0" ixz="0" iyy="${iyy}" iyz="0" izz="${izz}"/>
+	</inertial>
 </link>
 <joint  name="base_link_left_wheel" type="continuous">
@@ -49,4 +82,15 @@
 		</geometry>
 	</visual>
+	<collision>
+		<origin rpy="0 ${wheel_pitch} 0" xyz="0 0 0"/>
+		<geometry>
+			<cylinder length="${wheel_length}" radius="${wheel_radius}"/>
+		</geometry>
+	</collision>
+	<inertial>
+		<mass value="${mass}"/>
+		<origin xyz=" 0 0 0 "/>
+		<inertia ixx="${ixx}" ixy="0" ixz="0" iyy="${iyy}" iyz="0" izz="${izz}"/>
+	</inertial>
 </link>
 <joint  name="base_link_right_wheel" type="continuous">
@@ -64,4 +108,15 @@
 		</geometry>
 	</visual>
+	<collision>
+		<origin rpy="0 ${wheel_pitch} 0" xyz="0 0 0"/>
+		<geometry>
+			<sphere radius="${caster_radius}"/>
+		</geometry>
+	</collision>
+	<inertial>
+		<mass value="${mass}"/>
+		<origin xyz=" 0 0 0 "/>
+		<inertia ixx="${ixx}" ixy="0" ixz="0" iyy="${iyy}" iyz="0" izz="${izz}"/>
+	</inertial>
 </link>
 <joint name="base_link_caster" type="continuous">

Commit message: laser_scan_diff_drive

File: URDF/robot.xacro (robot description, xacro)
@@ -4,4 +4,7 @@
 <xacro:property name="base_link_length" value="0.02"/>
 <xacro:property name="base_link_radius" value="0.15"/>
+<!-- property of laser_scan-->
+<xacro:property name="joint_y_laser_scan" value="0.1"/>
+<xacro:property name="joint_z_laser_scan" value="0.03"/>
 <!-- property of wheel-->
 <xacro:property name="wheel_pitch" value="1.57"/>
@@ -24,4 +27,5 @@
 <xacro:property name="iyy" value="0.01"/>
 <xacro:property name="izz" value="0.01"/>
+<xacro:property name="laser_scan_length" value="0.04"/>
 <link name="dummy" >
 </link>
@@ -127,3 +131,68 @@
 	<limit effort="${effort}" velocity="${velocity}" lower="${lower}" upper="${upper}"/>
 </joint>
+<gazebo  reference="base_link">
+	<material>Gazebo/Black</material>
+	<turnGravityOff>false</turnGravityOff>
+</gazebo>
+<gazebo>
+	<plugin  name="differential_drive_robot" filename="libgazebo_ros_diff_drive.so">
+		<robotNamespace>/</robotNamespace>
+		<commandTopic>cmd_vel</commandTopic>
+		<odometryTopic>odom</odometryTopic>
+		<odometryFrame>odom</odometryFrame>
+		<robotBaseFrame>base_link</robotBaseFrame>
+		<publishWheelTF>false</publishWheelTF>
+		<publishOdomTF>true</publishOdomTF>
+		<publishWheelJointState>false</publishWheelJointState>
+		<legacyMode>true</legacyMode>
+		<wheelSeparation>${2*base_link_radius}</wheelSeparation>
+		<wheelDiameter>${2*wheel_radius}</wheelDiameter>
+		<wheelAcceleration>1.0</wheelAcceleration>
+		<wheelTorque>20.0</wheelTorque>
+		<updateRate>10.0</updateRate>
+		<leftJoint>base_link_left_wheel</leftJoint>
+		<rightJoint>base_link_right_wheel</rightJoint>
+	</plugin>
+</gazebo>
+<link name="laser_scan">
+	<visual>
+		<origin xyz="0 0 0" rpy="0 0 0"/>
+		<geometry>
+			<box size="${laser_scan_length} ${laser_scan_length} ${laser_scan_length}"/>
+		</geometry>
+	</visual>
+</link>
+<joint name="base_link_laser_scan" type="fixed">
+	<origin xyz="0 ${joint_y_laser_scan} ${joint_z_laser_scan}" rpy="0 0 0"/>
+	<parent link="base_link"/>
+	<child link="laser_scan"/>
+</joint>
+<gazebo reference="laser_scan">
+	<material>Gazebo/Red</material>
+	<turnGravityOff>false</turnGravityOff>
+	<sensor type="ray" name="laser_scan_sensor">
+		<pose>0 ${laser_scan_length/2} 0 0 0 0 </pose>
+		<visualize>true</visualize>
+		<update_rate>10.0</update_rate>
+		<ray>
+			<scan>
+				<horizontal>
+					<sample>1000</sample>
+					<resolution>1</resolution>
+					<min_angle>0</min_angle>
+					<max_angle>3.14</max_angle>
+				</horizontal>
+			</scan>
+			<range>
+				<min>0.1</min>
+				<max>10</max>
+				<resolution>1</resolution>
+			</range>
+		</ray>
+		<plugin name="lase_scanner" filename="libgazebo_ros_laser.so">
+			<topicName>/scan</topicName>
+			<frameName>laser_scan</frameName>
+		</plugin>
+	</sensor>
+</gazebo>
 </robot>

Commit message: navigation stack

File: URDF/robot.xacro (robot description, xacro)
@@ -133,5 +133,37 @@
 <gazebo  reference="base_link">
 	<material>Gazebo/Black</material>
-	<turnGravityOff>false</turnGravityOff>
+	<mu1 value="1.0"/>
+	<mu2 value="1.0"/>
+	<kp value="10000000.0" />
+	<kd value="1.0" />
+	<fdir1 value="1 0 0"/>
+    <turnGravityOff>false</turnGravityOff>
+</gazebo>
+<gazebo  reference="caster">
+	<material>Gazebo/Black</material>
+	<mu1 value="1.0"/>
+	<mu2 value="1.0"/>
+	<kp value="10000000.0" />
+	<kd value="1.0" />
+	<fdir1 value="1 0 0"/>
+    <turnGravityOff>false</turnGravityOff>
+</gazebo>
+<gazebo  reference="right_wheel">
+	<material>Gazebo/Black</material>
+	<mu1 value="1.0"/>
+	<mu2 value="1.0"/>
+	<kp value="10000000.0" />
+	<kd value="1.0" />
+	<fdir1 value="1 0 0"/>
+    <turnGravityOff>false</turnGravityOff>
+</gazebo>
+<gazebo  reference="left_wheel">
+	<material>Gazebo/Black</material>
+	<mu1 value="1.0"/>
+	<mu2 value="1.0"/>
+	<kp value="10000000.0" />
+	<kd value="1.0" />
+	<fdir1 value="1 0 0"/>
+    <turnGravityOff>false</turnGravityOff>
 </gazebo>
 <gazebo>
